Commit message: modify for eloquent

File: autocar2_bringup/urdf/autocar2.urdf (robot description, URDF)
Before this commit: robot turtlebot3_waffle, 13 links, 12 joints
Links:
- removed link base_footprint
- removed link camera_depth_frame
- removed link camera_depth_optical_frame
- removed link camera_link
- removed link camera_rgb_frame
- removed link camera_rgb_optical_frame
- removed link caster_back_left_link
- removed link caster_back_right_link
- removed link wheel_left_link
- removed link wheel_right_link
- added link horizontal_laser_link; visual cylinder length=0.05 radius=0.03
- added link vertical_laser_link; visual cylinder length=0.05 radius=0.03
- link base_link: mass 1.3729096e+00 -> None; geometry 
- link base_scan: mass 0.114 -> None; geometry visual cylinder length=0.05 radius=0.03
- link imu_link: geometry visual box size=0.06 0.04 0.02
Joints:
- removed joint base_joint
- removed joint camera_depth_joint
- removed joint camera_depth_optical_joint
- removed joint camera_joint
- removed joint camera_rgb_joint
- removed joint camera_rgb_optical_joint
- removed joint caster_back_left_joint
- removed joint caster_back_right_joint
- removed joint imu_joint
- removed joint scan_joint
- removed joint wheel_left_joint
- removed joint wheel_right_joint
- added joint horizontal_laser_link_joint: type fixed, parent base_link, child horizontal_laser_link, origin xyz=0.1007 0 0.0558
- added joint imu_link_joint: type fixed, parent base_link, child imu_link, origin xyz=0 0 0
- added joint laser_link_joint: type fixed, parent base_link, child base_scan, origin xyz=0.1007 0 0.2814 rpy=0 -1.570796 3.141593
- added joint vertical_laser_link_joint: type fixed, parent base_link, child vertical_laser_link, origin xyz=0.1007 0 0.1814 rpy=0 -1.570796 3.141593

Commit message: fix lua's odom option and urdf file

File: autocar2_bringup/urdf/autocar2.urdf (robot description, URDF)
Before this commit: robot turtlebot3_waffle, 13 links, 12 joints
Links:
- removed link base_scan
- added link laser_frame, mass 0.114; collision cylinder length=0.0315 radius=0.055; visual mesh filename=package://autocar2_bringup/meshes/sensors/lds.stl scale=0.001 0.001 0.001
Joints:
- joint scan_joint: child base_scan -> laser_frame

Commit message: fix urdf

File: autocar2_bringup/urdf/autocar2.urdf (robot description, URDF)
Before this commit: robot turtlebot3_waffle, 13 links, 12 joints
Links:
- removed link camera_depth_frame
- removed link camera_depth_optical_frame
- removed link camera_link
- removed link camera_rgb_frame
- removed link camera_rgb_optical_frame
- removed link caster_back_left_link
- removed link caster_back_right_link
- removed link wheel_left_link
- removed link wheel_right_link
- added link wheel1_link; visual cylinder length=0.015 radius=0.025
- added link wheel2_link; visual cylinder length=0.015 radius=0.025
- added link wheel3_link; visual cylinder length=0.015 radius=0.025
- added link wheel4_link; visual cylinder length=0.015 radius=0.025
- link base_footprint: geometry visual cylinder length=0.02 radius=0.03
- link base_link: mass 1.3729096e+00 -> None; geometry visual box size=0.1 0.2 0.05
- link imu_link: geometry visual box rpy=0.0 0.0 0.0 size=0.02 -0.02 0.02
- link laser_frame: mass 0.114 -> None; geometry visual cylinder length=0.02 radius=0.03
Joints:
- removed joint base_joint
- removed joint camera_depth_joint
- removed joint camera_depth_optical_joint
- removed joint camera_joint
- removed joint camera_rgb_joint
- removed joint camera_rgb_optical_joint
- removed joint caster_back_left_joint
- removed joint caster_back_right_joint
- removed joint imu_joint
- removed joint scan_joint
- removed joint wheel_left_joint
- removed joint wheel_right_joint
- added joint base_footprint_joint: type fixed, parent base_link, child base_footprint, origin xyz=0 0 0.025 rpy=0.0 0.0 0.0
- added joint imu_link_joint: type fixed, parent base_link, child imu_link, origin xyz=0 0 0
- added joint laser_joint: type fixed, parent base_link, child laser_frame, origin xyz=0 0 0.03 rpy=0.0 0.0 0.0
- added joint steering_joint1: type revolute, parent base_link, child wheel1_link, origin xyz=-0.057 0.06 -0.007 rpy=0.0 0.0 0.0, axis 0.0 0.0 1.0, limit lower=0 upper=0 effort=0 velocity=0
- added joint steering_joint2: type revolute, parent base_link, child wheel2_link, origin xyz=0.057 0.06 -0.007 rpy=0.0 0.0 0.0, axis 0.0 0.0 1.0, limit lower=0 upper=0 effort=0 velocity=0
- added joint wheel_joint1: type continuous, parent base_link, child wheel3_link, origin xyz=-0.057 -0.06 -0.007 rpy=0.0 0.0 0.0, axis 1.0 0.0 0.0
- added joint wheel_joint2: type continuous, parent base_link, child wheel4_link, origin xyz=0.057 -0.06 -0.007 rpy=0.0 0.0 0.0, axis 1.0 0.0 0.0
